Commit message: test martian

File: urdf/horse3d.urdf (robot description, URDF)
Before this commit: robot horse3d, 2 links, 1 joints
Links:
- removed link link1
- removed link link2
- added link body_link; collision sphere radius=0.2; visual sphere radius=0.2
- added link leg_link1; collision cylinder length=1.0 radius=0.1; visual cylinder length=1.0 radius=0.1
- added link leg_link2; collision cylinder length=1.0 radius=0.1; visual cylinder length=1.0 radius=0.1
- added link leg_link3; collision cylinder length=1.0 radius=0.1; visual cylinder length=1.0 radius=0.1
Joints:
- removed joint fixed
- added joint leg_joint1: type revolute, parent body_link, child leg_link1, origin xyz=0.0 0.0 0.0 rpy=0.0 0.0 0.0, axis 0 1 0, limit lower=-2.96705972839 upper=2.96705972839 effort=204 velocity=1.91986217719
- added joint leg_joint2: type revolute, parent body_link, child leg_link2, origin xyz=0.0 0.0 0.0 rpy=0.0 0.0 0.0, axis 0 0 1, limit lower=-2.96705972839 upper=2.96705972839 effort=204 velocity=1.91986217719
- added joint leg_joint3: type revolute, parent body_link, child leg_link3, origin xyz=0.0 0.0 0.0 rpy=0.0 0.0 0.0, axis 1 0 0, limit lower=-2.96705972839 upper=2.96705972839 effort=204 velocity=1.91986217719

Commit message: added svg of horse

File: urdf/horse3d.urdf (robot description, URDF)
Before this commit: robot test_robot, 4 links, 3 joints
Links:
- removed link body_link
- removed link leg_link1
- removed link leg_link2
- removed link leg_link3
- added link base_link; collision cylinder length=0.6 radius=0.2; visual cylinder length=0.6 radius=0.2
- added link right_leg; collision box size=0.6 0.1 -0.2; visual box size=0.6 0.1 0.2
Joints:
- removed joint leg_joint1
- removed joint leg_joint2
- removed joint leg_joint3
- added joint base_to_right_leg: type fixed, parent base_link, child right_leg, origin xyz=0.0 -0.22 0.25 rpy=0.0 0.0 0.0

Commit message: added body and foreleft leg

File: urdf/horse3d.urdf (robot description, URDF)
Before this commit: robot horse3d, 2 links, 1 joints
Links:
- removed link base_link
- removed link right_leg
- added link carpas_left; collision capsule length=0.235 radius=0.025; visual capsule length=0.235 radius=0.025
- added link carpas_left_vX
- added link carpas_left_vY
- added link coffin_foreleft; collision box size=0.11 0.078 0.048; visual box size=0.11 0.078 0.048
- added link humerus_left; collision capsule length=0.250 radius=0.033; visual capsule length=0.250 radius=0.033
- added link humerus_left_vX
- added link humerus_left_vY
- added link lumbar; collision sphere radius=0.095; visual sphere radius=0.095
- added link lumbar_vX
- added link lumbar_vY
- added link pastern_foreleft; collision capsule length=0.114 radius=0.02; visual capsule length=0.114 radius=0.02
- added link pastern_foreleft_vX
- added link pelvis; collision sphere radius=0.205; visual sphere radius=0.205
- added link pelvis_vX
- added link pelvis_vY
- added link radius_left; collision capsule length=0.370 radius=0.0375; visual capsule length=0.370 radius=0.0375
- added link scapula_left; collision capsule length=0.325 radius=0.0365; visual capsule length=0.325 radius=0.0365
- added link scapula_left_vX
- added link scapula_left_vY
- added link thoracic_back; collision sphere radius=0.22; visual sphere radius=0.22
- added link thoracic_front; collision sphere radius=0.245; visual sphere radius=0.245
Joints:
- removed joint base_to_right_leg
- added joint j_carpas_left_pitch: type revolute, parent carpas_left_vX, child carpas_left_vY, origin xyz=0.0 0 0.0 rpy=0.0 0.0 0.0, axis 0 1 0, limit lower=-1 upper=1 effort=0.0 velocity=0.0
- added joint j_carpas_left_roll: type revolute, parent radius_left, child carpas_left_vX, origin xyz=0.370 0 0.0 rpy=0.0 0.11 0.0, axis 1 0 0, limit lower=-1 upper=1 effort=0.0 velocity=0.0
- added joint j_carpas_left_yaw: type revolute, parent carpas_left_vY, child carpas_left, origin xyz=0.0 0 0.0 rpy=0.0 0.0 0.0, axis 0 0 1, limit lower=-1 upper=1 effort=0.0 velocity=0.0
- added joint j_coffin_foreleft: type revolute, parent pastern_foreleft, child coffin_foreleft, origin xyz=0.114 0 0.0 rpy=0.0 -1.04 0.0, axis 0 1 0, limit lower=-1 upper=1 effort=0.0 velocity=0.0
- added joint j_humerus_left_pitch: type revolute, parent humerus_left_vX, child humerus_left_vY, origin xyz=0.0 0 0.0 rpy=0.0 0.0 0.0, axis 0 1 0, limit lower=-1 upper=1 effort=0.0 velocity=0.0
- added joint j_humerus_left_roll: type revolute, parent scapula_left, child humerus_left_vX, origin xyz=0.325 0 0.0 rpy=0.0 1.3148 0.0, axis 1 0 0, limit lower=-1 upper=1 effort=0.0 velocity=0.0
- added joint j_humerus_left_yaw: type revolute, parent humerus_left_vY, child humerus_left, origin xyz=0.0 0 0.0 rpy=0.0 0.0 0.0, axis 0 0 1, limit lower=-1 upper=1 effort=0.0 velocity=0.0
- added joint j_lumbar_pitch: type revolute, parent lumbar_vX, child lumbar_vY, origin xyz=0.0 0 0.0 rpy=0.0 0.0 0.0, axis 0 1 0, limit lower=-1 upper=1 effort=0.0 velocity=0.0
- added joint j_lumbar_roll: type revolute, parent thoracic_back, child lumbar_vX, origin xyz=-0.30 0 0.17 rpy=0.0 0.0 0.0, axis 1 0 0, limit lower=-1 upper=1 effort=0.0 velocity=0.0
- added joint j_lumbar_yaw: type revolute, parent lumbar_vY, child lumbar, origin xyz=0.0 0 0.0 rpy=0.0 0.0 0.0, axis 0 0 1, limit lower=-1 upper=1 effort=0.0 velocity=0.0
- added joint j_pastern_foreleft_pitch: type revolute, parent pastern_foreleft_vX, child pastern_foreleft, origin xyz=0.0 0 0.0 rpy=0.0 0.0 0.0, axis 0 1 0, limit lower=-1 upper=1 effort=0.0 velocity=0.0
- added joint j_pastern_foreleft_roll: type revolute, parent carpas_left, child pastern_foreleft_vX, origin xyz=0.235 0 0.0 rpy=0.0 -0.582 0.0, axis 1 0 0, limit lower=-1 upper=1 effort=0.0 velocity=0.0
- added joint j_pelvis_pitch: type revolute, parent pelvis_vX, child pelvis_vY, origin xyz=0.0 0 0.0 rpy=0.0 0.0 0.0, axis 0 1 0, limit lower=-1 upper=1 effort=0.0 velocity=0.0
- added joint j_pelvis_roll: type revolute, parent lumbar, child pelvis_vX, origin xyz=-0.178 0 0.013 rpy=0.0 0.0 0.0, axis 1 0 0, limit lower=-1 upper=1 effort=0.0 velocity=0.0
- added joint j_pelvis_yaw: type revolute, parent pelvis_vY, child pelvis, origin xyz=0.0 0 0.0 rpy=0.0 0.0 0.0, axis 0 0 1, limit lower=-1 upper=1 effort=0.0 velocity=0.0
- added joint j_radius_left: type revolute, parent humerus_left, child radius_left, origin xyz=0.250 0 0.0 rpy=0.0 -0.6291 0.0, axis 0 1 0, limit lower=-1 upper=1 effort=0.0 velocity=0.0
- added joint j_scapula_left_pitch: type revolute, parent scapula_left_vX, child scapula_left_vY, origin xyz=0.0 0 0.0 rpy=0.0 0.0 0.0, axis 0 1 0, limit lower=-1 upper=1 effort=0.0 velocity=0.0
- added joint j_scapula_left_roll: type revolute, parent thoracic_front, child scapula_left_vX, origin xyz=0.0164 0.145 0.222 rpy=0.0 0.825 0.0, axis 1 0 0, limit lower=-1 upper=1 effort=0.0 velocity=0.0
- added joint j_scapula_left_yaw: type revolute, parent scapula_left_vY, child scapula_left, origin xyz=0.0 0 0.0 rpy=0.0 0.0 0.0, axis 0 0 1, limit lower=-1 upper=1 effort=0.0 velocity=0.0
- added joint j_thoracic: type fixed, parent thoracic_front, child thoracic_back, origin xyz=-0.18 0 0 rpy=0.0 0.0 0.0

Commit message: added whole body

File: urdf/horse3d.urdf (robot description, URDF)
Before this commit: robot horse3d, 21 links, 20 joints
Links:
- added link carpas_right; collision capsule length=0.235 radius=0.025; visual capsule length=0.235 radius=0.025
- added link carpas_right_vX
- added link carpas_right_vY
- added link coffin_foreright; collision box size=0.11 0.078 0.048; visual box size=0.11 0.078 0.048
- added link coffin_hindleft; collision box size=0.11 0.078 0.048; visual box size=0.11 0.078 0.048
- added link coffin_hindright; collision box size=0.11 0.078 0.048; visual box size=0.11 0.078 0.048
- added link femur_left; collision capsule length=0.306 radius=0.040; visual capsule length=0.306 radius=0.040
- added link femur_left_vX
- added link femur_left_vY
- added link femur_right; collision capsule length=0.306 radius=0.040; visual capsule length=0.306 radius=0.040
- added link femur_right_vX
- added link femur_right_vY
- added link head; collision box size=0.4419 0.1861 0.2474; visual box size=0.4419 0.1861 0.2474
- added link head_vX
- added link head_vY
- added link humerus_right; collision capsule length=0.250 radius=0.033; visual capsule length=0.250 radius=0.033
- added link humerus_right_vX
- added link humerus_right_vY
- added link neck; collision capsule length=0.443 radius=0.05; visual capsule length=0.443 radius=0.05
- added link neck_vX
- added link neck_vY
- added link pastern_foreright; collision capsule length=0.114 radius=0.02; visual capsule length=0.114 radius=0.02
- added link pastern_foreright_vX
- added link pastern_hindleft; collision capsule length=0.11 radius=0.02; visual capsule length=0.11 radius=0.02
- added link pastern_hindleft_vX
- added link pastern_hindright; collision capsule length=0.11 radius=0.02; visual capsule length=0.11 radius=0.02
- added link pastern_hindright_vX
- added link radius_right; collision capsule length=0.370 radius=0.0375; visual capsule length=0.370 radius=0.0375
- added link scapula_right; collision capsule length=0.325 radius=0.0365; visual capsule length=0.325 radius=0.0365
- added link scapula_right_vX
- added link scapula_right_vY
- added link tail_back; collision capsule length=0.245 radius=0.026; visual capsule length=0.245 radius=0.026
- added link tail_back_vX
- added link tail_front; collision capsule length=0.245 radius=0.026; visual capsule length=0.245 radius=0.026
- added link tail_front_vX
- added link tarsal_left; collision capsule length=0.26 radius=0.021; visual capsule length=0.26 radius=0.021
- added link tarsal_left_vX
- added link tarsal_left_vY
- added link tarsal_right; collision capsule length=0.26 radius=0.021; visual capsule length=0.26 radius=0.021
- added link tarsal_right_vX
- added link tarsal_right_vY
- added link tibia_left; collision capsule length=0.36 radius=0.030; visual capsule length=0.36 radius=0.030
- added link tibia_right; collision capsule length=0.36 radius=0.030; visual capsule length=0.36 radius=0.030
Joints:
- added joint j_carpas_right_pitch: type revolute, parent carpas_right_vX, child carpas_right_vY, origin xyz=0.0 0 0.0 rpy=0.0 0.0 0.0, axis 0 1 0, limit lower=0. upper=0.8 effort=0.0 velocity=0.0
- added joint j_carpas_right_roll: type revolute, parent radius_right, child carpas_right_vX, origin xyz=0.370 0 0.0 rpy=0.0 0.11 0.0, axis 1 0 0, limit lower=-0.05 upper=0.05 effort=0.0 velocity=0.0
- added joint j_carpas_right_yaw: type revolute, parent carpas_right_vY, child carpas_right, origin xyz=0.0 0 0.0 rpy=0.0 0.0 0.0, axis 0 0 1, limit lower=-0.05 upper=0.05 effort=0.0 velocity=0.0
- added joint j_coffin_foreright: type revolute, parent pastern_foreright, child coffin_foreright, origin xyz=0.114 0 0.0 rpy=0.0 -1.04 0.0, axis 0 1 0, limit lower=-0.1 upper=0.1 effort=0.0 velocity=0.0
- added joint j_coffin_hindleft: type revolute, parent pastern_hindleft, child coffin_hindleft, origin xyz=0.114 0 0.0 rpy=0.0 -1.03 0.0, axis 0 1 0, limit lower=-0.1 upper=0.1 effort=0.0 velocity=0.0
- added joint j_coffin_hindright: type revolute, parent pastern_hindright, child coffin_hindright, origin xyz=0.114 0 0.0 rpy=0.0 -1.03 0.0, axis 0 1 0, limit lower=-0.1 upper=0.1 effort=0.0 velocity=0.0
- added joint j_femur_left_pitch: type revolute, parent femur_left_vX, child femur_left_vY, origin xyz=0.0 0 0.0 rpy=0.0 0.0 0.0, axis 0 1 0, limit lower=-0.5 upper=1 effort=0.0 velocity=0.0
- added joint j_femur_left_roll: type revolute, parent pelvis, child femur_left_vX, origin xyz=-0.1935 0.189 -0.14705 rpy=0.0 1.2726 0.0, axis 1 0 0, limit lower=-0.1 upper=0.1 effort=0.0 velocity=0.0
- added joint j_femur_left_yaw: type revolute, parent femur_left_vY, child femur_left, origin xyz=0.0 0 0.0 rpy=0.0 0.0 0.0, axis 0 0 1, limit lower=-0.1 upper=0.1 effort=0.0 velocity=0.0
- added joint j_femur_right_pitch: type revolute, parent femur_right_vX, child femur_right_vY, origin xyz=0.0 0 0.0 rpy=0.0 0.0 0.0, axis 0 1 0, limit lower=-0.5 upper=1 effort=0.0 velocity=0.0
- added joint j_femur_right_roll: type revolute, parent pelvis, child femur_right_vX, origin xyz=-0.1935 -0.189 -0.14705 rpy=0.0 1.2726 0.0, axis 1 0 0, limit lower=-0.1 upper=0.1 effort=0.0 velocity=0.0
- added joint j_femur_right_yaw: type revolute, parent femur_right_vY, child femur_right, origin xyz=0.0 0 0.0 rpy=0.0 0.0 0.0, axis 0 0 1, limit lower=-0.1 upper=0.1 effort=0.0 velocity=0.0
- added joint j_head_pitch: type revolute, parent head_vX, child head_vY, origin xyz=0.0 0 0.0 rpy=0.0 0.0 0.0, axis 0 1 0, limit lower=-0.5 upper=0.5 effort=0.0 velocity=0.0
- added joint j_head_roll: type revolute, parent neck, child head_vX, origin xyz=0.443 0 0.0 rpy=0.0 1.8567 0.0, axis 1 0 0, limit lower=-0.1 upper=0.1 effort=0.0 velocity=0.0
- added joint j_head_yaw: type revolute, parent head_vY, child head, origin xyz=0.0 0 0.0 rpy=0.0 0.0 0.0, axis 0 0 1, limit lower=-0.5 upper=0.5 effort=0.0 velocity=0.0
- added joint j_humerus_right_pitch: type revolute, parent humerus_right_vX, child humerus_right_vY, origin xyz=0.0 0 0.0 rpy=0.0 0.0 0.0, axis 0 1 0, limit lower=-0.7 upper=0.2 effort=0.0 velocity=0.0
- added joint j_humerus_right_roll: type revolute, parent scapula_right, child humerus_right_vX, origin xyz=0.325 0 0.0 rpy=0.0 1.3148 0.0, axis 1 0 0, limit lower=-0.1 upper=0.1 effort=0.0 velocity=0.0
- added joint j_humerus_right_yaw: type revolute, parent humerus_right_vY, child humerus_right, origin xyz=0.0 0 0.0 rpy=0.0 0.0 0.0, axis 0 0 1, limit lower=-0.1 upper=0.1 effort=0.0 velocity=0.0
- added joint j_neck_pitch: type revolute, parent neck_vX, child neck_vY, origin xyz=0.0 0 0.0 rpy=0.0 0.0 0.0, axis 0 1 0, limit lower=-0.5 upper=0.5 effort=0.0 velocity=0.0
- added joint j_neck_roll: type revolute, parent thoracic_front, child neck_vX, origin xyz=0.201 0 0.130 rpy=0.0 -1.0 0.0, axis 1 0 0, limit lower=-0.5 upper=0.5 effort=0.0 velocity=0.0
- added joint j_neck_yaw: type revolute, parent neck_vY, child neck, origin xyz=0.0 0 0.0 rpy=0.0 0.0 0.0, axis 0 0 1, limit lower=-0.5 upper=0.5 effort=0.0 velocity=0.0
- added joint j_pastern_foreright_pitch: type revolute, parent pastern_foreright_vX, child pastern_foreright, origin xyz=0.0 0 0.0 rpy=0.0 0.0 0.0, axis 0 1 0, limit lower=-0.5 upper=1 effort=0.0 velocity=0.0
- added joint j_pastern_foreright_roll: type revolute, parent carpas_right, child pastern_foreright_vX, origin xyz=0.235 0 0.0 rpy=0.0 -0.582 0.0, axis 1 0 0, limit lower=-0.1 upper=0.1 effort=0.0 velocity=0.0
- added joint j_pastern_hindleft_pitch: type revolute, parent pastern_hindleft_vX, child pastern_hindleft, origin xyz=0.0 0 0.0 rpy=0.0 0.0 0.0, axis 0 1 0, limit lower=-0.5 upper=1 effort=0.0 velocity=0.0
- added joint j_pastern_hindleft_roll: type revolute, parent tarsal_left, child pastern_hindleft_vX, origin xyz=0.26 0 0.0 rpy=0.0 -0.582 0.0, axis 1 0 0, limit lower=-0.1 upper=0.1 effort=0.0 velocity=0.0
- added joint j_pastern_hindright_pitch: type revolute, parent pastern_hindright_vX, child pastern_hindright, origin xyz=0.0 0 0.0 rpy=0.0 0.0 0.0, axis 0 1 0, limit lower=-0.5 upper=1 effort=0.0 velocity=0.0
- added joint j_pastern_hindright_roll: type revolute, parent tarsal_right, child pastern_hindright_vX, origin xyz=0.26 0 0.0 rpy=0.0 -0.582 0.0, axis 1 0 0, limit lower=-0.1 upper=0.1 effort=0.0 velocity=0.0
- added joint j_radius_right: type revolute, parent humerus_right, child radius_right, origin xyz=0.250 0 0.0 rpy=0.0 -0.6291 0.0, axis 0 1 0, limit lower=-0.6 upper=0.6 effort=0.0 velocity=0.0
- added joint j_scapula_right_pitch: type revolute, parent scapula_right_vX, child scapula_right_vY, origin xyz=0.0 0 0.0 rpy=0.0 0.0 0.0, axis 0 1 0, limit lower=-0.2 upper=0.2 effort=0.0 velocity=0.0
- added joint j_scapula_right_roll: type revolute, parent thoracic_front, child scapula_right_vX, origin xyz=0.0164 -0.145 0.222 rpy=0.0 0.825 0.0, axis 1 0 0, limit lower=-0.2 upper=0.2 effort=0.0 velocity=0.0
- added joint j_scapula_right_yaw: type revolute, parent scapula_right_vY, child scapula_right, origin xyz=0.0 0 0.0 rpy=0.0 0.0 0.0, axis 0 0 1, limit lower=-0.1 upper=0.1 effort=0.0 velocity=0.0
- added joint j_tail_back_pitch: type revolute, parent tail_front, child tail_back_vX, origin xyz=0.245 0 0.0 rpy=0.0 -0.3935 0.0, axis 0 1 0, limit lower=-1 upper=1 effort=0.0 velocity=0.0
- added joint j_tail_back_yaw: type revolute, parent tail_back_vX, child tail_back, origin xyz=0.0 0 0.0 rpy=0.0 0.0 0.0, axis 0 0 1, limit lower=-1 upper=1 effort=0.0 velocity=0.0
- added joint j_tail_front_pitch: type revolute, parent pelvis, child tail_front_vX, origin xyz=-0.259 0 0.0314 rpy=0.0 2.6 0.0, axis 0 1 0, limit lower=-1 upper=1 effort=0.0 velocity=0.0
- added joint j_tail_front_yaw: type revolute, parent tail_front_vX, child tail_front, origin xyz=0.0 0 0.0 rpy=0.0 0.0 0.0, axis 0 0 1, limit lower=-1 upper=1 effort=0.0 velocity=0.0
- added joint j_tarsal_left_pitch: type revolute, parent tarsal_left_vX, child tarsal_left_vY, origin xyz=0.0 0 0.0 rpy=0.0 0.0 0.0, axis 0 1 0, limit lower=-0.5 upper=0.5 effort=0.0 velocity=0.0
- added joint j_tarsal_left_roll: type revolute, parent tibia_left, child tarsal_left_vX, origin xyz=0.36, 0, 0.0 rpy=0.0 -0.47825 0.0, axis 1 0 0, limit lower=-0.1 upper=0.1 effort=0.0 velocity=0.0
- added joint j_tarsal_left_yaw: type revolute, parent tarsal_left_vY, child tarsal_left, origin xyz=0.0 0 0.0 rpy=0.0 0.0 0.0, axis 0 0 1, limit lower=-0.1 upper=0.1 effort=0.0 velocity=0.0
- added joint j_tarsal_right_pitch: type revolute, parent tarsal_right_vX, child tarsal_right_vY, origin xyz=0.0 0 0.0 rpy=0.0 0.0 0.0, axis 0 1 0, limit lower=-0.5 upper=0.5 effort=0.0 velocity=0.0
- added joint j_tarsal_right_roll: type revolute, parent tibia_right, child tarsal_right_vX, origin xyz=0.36, 0, 0.0 rpy=0.0 -0.47825 0.0, axis 1 0 0, limit lower=-0.1 upper=0.1 effort=0.0 velocity=0.0
- added joint j_tarsal_right_yaw: type revolute, parent tarsal_right_vY, child tarsal_right, origin xyz=0.0 0 0.0 rpy=0.0 0.0 0.0, axis 0 0 1, limit lower=-0.1 upper=0.1 effort=0.0 velocity=0.0
- added joint j_tibia_left: type revolute, parent femur_left, child tibia_left, origin xyz=0.306, 0, 0.0 rpy=0.0 0.80176, 0.0, axis 0 1 0, limit lower=-0.5 upper=0.5 effort=0.0 velocity=0.0
- added joint j_tibia_right: type revolute, parent femur_right, child tibia_right, origin xyz=0.306, 0, 0.0 rpy=0.0 0.80176, 0.0, axis 0 1 0, limit lower=-0.5 upper=0.5 effort=0.0 velocity=0.0
- joint j_carpas_left_pitch: limit lower=-1 upper=1 effort=0.0 velocity=0.0 -> lower=0. upper=0.8 effort=0.0 velocity=0.0
- joint j_carpas_left_roll: limit lower=-1 upper=1 effort=0.0 velocity=0.0 -> lower=-0.05 upper=0.05 effort=0.0 velocity=0.0
- joint j_carpas_left_yaw: limit lower=-1 upper=1 effort=0.0 velocity=0.0 -> lower=-0.05 upper=0.05 effort=0.0 velocity=0.0
- joint j_coffin_foreleft: limit lower=-1 upper=1 effort=0.0 velocity=0.0 -> lower=-0.1 upper=0.1 effort=0.0 velocity=0.0
- joint j_humerus_left_pitch: limit lower=-1 upper=1 effort=0.0 velocity=0.0 -> lower=-0.7 upper=0.2 effort=0.0 velocity=0.0
- joint j_humerus_left_roll: limit lower=-1 upper=1 effort=0.0 velocity=0.0 -> lower=-0.1 upper=0.1 effort=0.0 velocity=0.0
- joint j_humerus_left_yaw: limit lower=-1 upper=1 effort=0.0 velocity=0.0 -> lower=-0.1 upper=0.1 effort=0.0 velocity=0.0
- joint j_lumbar_pitch: limit lower=-1 upper=1 effort=0.0 velocity=0.0 -> lower=-0.2 upper=0.2 effort=0.0 velocity=0.0
- joint j_lumbar_roll: limit lower=-1 upper=1 effort=0.0 velocity=0.0 -> lower=-0.2 upper=0.2 effort=0.0 velocity=0.0
- joint j_lumbar_yaw: limit lower=-1 upper=1 effort=0.0 velocity=0.0 -> lower=-0.2 upper=0.2 effort=0.0 velocity=0.0
- joint j_pastern_foreleft_pitch: limit lower=-1 upper=1 effort=0.0 velocity=0.0 -> lower=-0.5 upper=1 effort=0.0 velocity=0.0
- joint j_pastern_foreleft_roll: limit lower=-1 upper=1 effort=0.0 velocity=0.0 -> lower=-0.1 upper=0.1 effort=0.0 velocity=0.0
- joint j_pelvis_pitch: limit lower=-1 upper=1 effort=0.0 velocity=0.0 -> lower=-0.2 upper=0.2 effort=0.0 velocity=0.0
- joint j_pelvis_roll: limit lower=-1 upper=1 effort=0.0 velocity=0.0 -> lower=-0.2 upper=0.2 effort=0.0 velocity=0.0
- joint j_pelvis_yaw: limit lower=-1 upper=1 effort=0.0 velocity=0.0 -> lower=-0.2 upper=0.2 effort=0.0 velocity=0.0
- joint j_radius_left: limit lower=-1 upper=1 effort=0.0 velocity=0.0 -> lower=-0.6 upper=0.6 effort=0.0 velocity=0.0
- joint j_scapula_left_pitch: limit lower=-1 upper=1 effort=0.0 velocity=0.0 -> lower=-0.2 upper=0.2 effort=0.0 velocity=0.0
- joint j_scapula_left_roll: limit lower=-1 upper=1 effort=0.0 velocity=0.0 -> lower=-0.2 upper=0.2 effort=0.0 velocity=0.0
- joint j_scapula_left_yaw: limit lower=-1 upper=1 effort=0.0 velocity=0.0 -> lower=-0.1 upper=0.1 effort=0.0 velocity=0.0
